File: hardware/atf1502as-tqfp44-board/neogeo-diag-aes-cha-atf1502as-tqfp44.kicad_sch (KiCad schematic)
At the start: 18 parts, among them J1 neogeo-aes-cha-a-side-edge, J2 neogeo-aes-cha-a-side-edge, J3 neogeo-aes-cha-b-side-edge, J4 neogeo-aes-cha-b-side-edge, J5 JTAG, U1 74HC574, U2 ATF1502AS-xAx44, U3 74HC574, U4 27C010 / 27C1001, U5 27C010 / 27C1001

Commit message: Minor tweaks, Bump revision number on all boards so they are the same
Changed lines of the file:
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@@
     (effects (font (size 3 3)) (justify left bottom))
   )
-  (text "M1 ROM + Address Logic" (at 278.765 146.685 0)
+  (text "M1 ROM + Address Logic" (at 286.385 146.685 0)
     (effects (font (size 3 3)) (justify left bottom))
   )
